Commit message: Allegro: 60 deg mount yaw, and extend the fingers at the home pose
Both changes come from looking at the hand in the reachability viewer.

**Mount yaw 60 deg CCW.** Set as the DEFAULT in build_allegro_urdf.py, not just
a CLI flag: rebuilding the URDF without arguments must reproduce the shipped
robot, or the hand silently reverts to 0 and invalidates any policy trained
against it. Unlike the mount z offset, which is derived (0.071 - 0.045, the
difference between the two arms' flange-to-ee distances), the yaw is a judgement
about how the hand presents itself to the table and is recorded as such.

**Fingers extended at home.** Allegro was using Isaac Lab's KUKA_ALLEGRO_CFG
pose, in which 13 of 16 hand joints are non-zero -- each finger curled ~52 deg,
the three flexion joints sitting at 0.3 rad (29% into their range). SHARPA's
home is all-zeros, which for its flexion joints (lower limit 0.0) is the hard
extension stop. So the two hands were starting episodes at different points in
their own ranges, which changes how quickly each can enclose an object. That is
a config choice, not a hardware property, and it would have leaked straight into
the comparison.

The fingers now start straight. The thumb cannot follow the same rule:
thumb_joint_0 has limits [0.279, 1.571], so 0.0 is outside its range entirely
and would be clamped -- Allegro's zero is simply not SHARPA's zero. Its neutral
is defined by its own range, so it keeps Isaac Lab's 1.5 (95% of range), which
opposes the thumb across the fingers, the analogue of where SHARPA's thumb
already sits at zero.

After the change the two hands line up closely at home: fingertip centroid in
the shared iiwa14_link_7 frame is z = 0.2507 (SHARPA) vs 0.2546 (Allegro).

Co-Authored-By: Claude Opus 5 (1M context) <noreply@anthropic.com>

File: assets/urdf/kuka_allegro_iiwa14_description/iiwa14_allegro.urdf (robot description, URDF)
Before this commit: robot iiwa14_allegro, 27 links, 26 joints
Joints:
- joint iiwa14_allegro: origin xyz=0 0 0.025999999999999995 rpy=0 0 0.0 -> xyz=0 0 0.025999999999999995 rpy=0 0 1.0471975511965976

Commit message: Allegro becomes a LEFT hand, thumb spread at home, mount yaw 150 deg
**Handedness.** SHARPA is a left hand; the stock Allegro asset is right-handed,
which made the two robots differ in more than the hand under test. The builder
now mirrors the hand subtree about its mount's y=0 plane by default.

The asset's own comment claims a left hand only needs each finger's y offset and
splay angle negated. That is incomplete, and measurably so -- reflecting the
meshes about y leaves a residual of 34.8 mm max on the palm (base_link.obj) and
30.3 mm on thumb_base.obj, while the finger links are genuinely symmetric
(0.04 mm). Following the comment alone would produce left-hand kinematics
wearing a right-hand palm. So the builder applies the full reflection
M = diag(1,-1,1): origins, rotations (R -> M R M, still a rotation since
det = 1), revolute axes (a -> -M a, the extra sign because an axis is a
pseudovector and it keeps a positive joint angle meaning the same motion, which
matters with asymmetric limits), and mirrored copies of every hand mesh with
reversed winding.

Verified against the right-hand build: max |left_pos - mirror(right_pos)| is
1 micron over 6 random configurations x 5 links, that being %.9g write-out
round-off. Finger y-order inverts exactly (index -0.0363 -> +0.0363,
ring +0.0539 -> -0.0539).

**Home pose**: thumb_joint_0 goes to its lower limit 0.279244444444 -- abducted
out alongside the fingers, hand wide open -- chosen visually against how SHARPA
presents itself at its own all-zeros home. Fingertip pad offsets are re-measured
on the mirrored meshes, so their y is negated.

**Mount yaw 150 deg**, also chosen visually. Note the two interact: mirroring
inverts the sense of this rotation, so a yaw picked on the right-hand asset does
not carry over. Recorded in the builder so it is re-checked after any handedness
change.

Co-Authored-By: Claude Opus 5 (1M context) <noreply@anthropic.com>

File: assets/urdf/kuka_allegro_iiwa14_description/iiwa14_allegro.urdf (robot description, URDF)
Before this commit: robot iiwa14_allegro, 27 links, 26 joints
Links:
- link allegro_mount: geometry collision mesh filename=allegro_meshes_mirrored/allegro_meshes__mounts__allegro_mou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; visual mesh filename=allegro_meshes_mirrored/allegro_meshes__mounts__allegro_mou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
- link index_link_0: geometry collision mesh filename=allegro_meshes_mirrored/allegro_meshes__allegro__primary_ba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; visual mesh filename=allegro_meshes_mirrored/allegro_meshes__allegro__primary_ba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
- link index_link_1: geometry collision mesh filename=allegro_meshes_mirrored/allegro_meshes__allegro__primary_pr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; visual mesh filename=allegro_meshes_mirrored/allegro_meshes__allegro__primary_pr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
- link index_link_2: geometry collision mesh filename=allegro_meshes_mirrored/allegro_meshes__allegro__primary_me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; visual mesh filename=allegro_meshes_mirrored/allegro_meshes__allegro__primary_me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
- link index_link_3: geometry collision mesh filename=allegro_meshes_mirrored/allegro_meshes__biotac__biotac_sens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; visual mesh filename=allegro_meshes_mirrored/allegro_meshes__biotac__biotac_sens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
- link middle_link_0: geometry collision mesh filename=allegro_meshes_mirrored/allegro_meshes__allegro__primary_ba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; visual mesh filename=allegro_meshes_mirrored/allegro_meshes__allegro__primary_ba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
- link middle_link_1: geometry collision mesh filename=allegro_meshes_mirrored/allegro_meshes__allegro__primary_pr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; visual mesh filename=allegro_meshes_mirrored/allegro_meshes__allegro__primary_pr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
- link middle_link_2: geometry collision mesh filename=allegro_meshes_mirrored/allegro_meshes__allegro__primary_me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; visual mesh filename=allegro_meshes_mirrored/allegro_meshes__allegro__primary_me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
- link middle_link_3: geometry collision mesh filename=allegro_meshes_mirrored/allegro_meshes__biotac__biotac_sens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; visual mesh filename=allegro_meshes_mirrored/allegro_meshes__biotac__biotac_sens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
- link palm_link: geometry collision mesh filename=allegro_meshes_mirrored/allegro_meshes__allegro__base_link.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; visual mesh filename=allegro_meshes_mirrored/allegro_meshes__allegro__base_link.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
- link ring_link_0: geometry collision mesh filename=allegro_meshes_mirrored/allegro_meshes__allegro__primary_ba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; visual mesh filename=allegro_meshes_mirrored/allegro_meshes__allegro__primary_ba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
- link ring_link_1: geometry collision mesh filename=allegro_meshes_mirrored/allegro_meshes__allegro__primary_pr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; visual mesh filename=allegro_meshes_mirrored/allegro_meshes__allegro__primary_pr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
- link ring_link_2: geometry collision mesh filename=allegro_meshes_mirrored/allegro_meshes__allegro__primary_me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; visual mesh filename=allegro_meshes_mirrored/allegro_meshes__allegro__primary_me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
- link ring_link_3: geometry collision mesh filename=allegro_meshes_mirrored/allegro_meshes__biotac__biotac_sens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; visual mesh filename=allegro_meshes_mirrored/allegro_meshes__biotac__biotac_sens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
- link thumb_link_0: geometry collision mesh filename=allegro_meshes_mirrored/allegro_meshes__allegro__thumb_base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; visual mesh filename=allegro_meshes_mirrored/allegro_meshes__allegro__thumb_base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
- link thumb_link_1: geometry collision mesh filename=allegro_meshes_mirrored/allegro_meshes__allegro__thumb_prox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; visual mesh filename=allegro_meshes_mirrored/allegro_meshes__allegro__thumb_prox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
- link thumb_link_2: geometry collision mesh filename=allegro_meshes_mirrored/allegro_meshes__allegro__thumb_medi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; visual mesh filename=allegro_meshes_mirrored/allegro_meshes__allegro__thumb_medi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
- link thumb_link_3: geometry collision mesh filename=allegro_meshes_mirrored/allegro_meshes__biotac__biotac_sens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; visual mesh filename=allegro_meshes_mirrored/allegro_meshes__biotac__biotac_sens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
Joints:
- joint allegro_mount_joint: origin xyz=0.008219 -0.02063 0.08086 rpy=0 -1.5708 0.785398 -> xyz=0.008219 0.02063 0.08086 rpy=-0.785398 -1.57079265 0
- joint iiwa14_allegro: origin xyz=0 0 0.025999999999999995 rpy=0 0 1.0471975511965976 -> xyz=0 0 0.025999999999999995 rpy=0 0 2.6179938779914944
- joint index_joint_0: axis 0 0 1 -> -0 -0 -1; origin xyz=0.0514302 -0.03632 -0.0113 rpy=3.1415 -1.57075 -0.0872638888889 -> xyz=0.0514302 0.03632 -0.0113 rpy=-3.1415 -1.57075 0.0872638889
- joint index_joint_1: axis 0 0 1 -> -0 -0 -1; origin xyz=0.0 0.0 0.0 rpy=3.1415 -1.57075 1.57075 -> xyz=0 0 0 rpy=-3.1415 -1.57075 -1.57075
- joint index_joint_2: axis 0 0 1 -> -0 -0 -1; origin xyz=0.054 0.0 0.0 rpy=0.0 0.0 0.0 -> xyz=0.054 0 0 rpy=0 -0 0
- joint index_joint_3: axis 0 0 1 -> -0 -0 -1; origin xyz=0.0384 0.0 0.0 rpy=0.0 0.0 0.0 -> xyz=0.0384 0 0 rpy=0 -0 0
- joint middle_joint_0: axis 0 0 1 -> -0 -0 -1; origin xyz=0.0537375 0.0087771 -0.0113 rpy=3.1415 -1.57075 0 -> xyz=0.0537375 -0.0087771 -0.0113 rpy=-3.1415 -1.57075 0
- joint middle_joint_1: axis 0 0 1 -> -0 -0 -1; origin xyz=0.0 0.0 0.0 rpy=3.1415 -1.57075 1.57075 -> xyz=0 0 0 rpy=-3.1415 -1.57075 -1.57075
- joint middle_joint_2: axis 0 0 1 -> -0 -0 -1; origin xyz=0.054 0.0 0.0 rpy=0.0 0.0 0.0 -> xyz=0.054 0 0 rpy=0 -0 0
- joint middle_joint_3: axis 0 0 1 -> -0 -0 -1; origin xyz=0.0384 0.0 0.0 rpy=0.0 0.0 0.0 -> xyz=0.0384 0 0 rpy=0 -0 0
- joint ring_joint_0: axis 0 0 1 -> -0 -0 -1; origin xyz=0.0514302 0.0538749 -0.0113 rpy=3.1415 -1.57075 0.0872638888889 -> xyz=0.0514302 -0.0538749 -0.0113 rpy=-3.1415 -1.57075 -0.0872638889
- joint ring_joint_1: axis 0 0 1 -> -0 -0 -1; origin xyz=0.0 0.0 0.0 rpy=3.1415 -1.57075 1.57075 -> xyz=0 0 0 rpy=-3.1415 -1.57075 -1.57075
- joint ring_joint_2: axis 0 0 1 -> -0 -0 -1; origin xyz=0.054 0.0 0.0 rpy=0.0 0.0 0.0 -> xyz=0.054 0 0 rpy=0 -0 0
- joint ring_joint_3: axis 0 0 1 -> -0 -0 -1; origin xyz=0.0384 0.0 0.0 rpy=0.0 0.0 0.0 -> xyz=0.0384 0 0 rpy=0 -0 0
- joint thumb_joint_0: axis 0 0 1 -> -0 -0 -1; origin xyz=-0.0367482 -0.0081281 -0.0295 rpy=-1.57075 -1.57075 1.48348611111 -> xyz=-0.0367482 0.0081281 -0.0295 rpy=1.57075 -1.57075 -1.48348611
- joint thumb_joint_1: axis 0 0 1 -> -0 -0 -1; origin xyz=0.005 0.0 0.0 rpy=1.57075 0 0 -> xyz=0.005 0 0 rpy=-1.57075 -0 0
- joint thumb_joint_2: axis 0 0 1 -> -0 -0 -1; origin xyz=0 0 0.0554 rpy=3.1415 -1.57075 0.0 -> xyz=0 0 0.0554 rpy=-3.1415 -1.57075 0
- joint thumb_joint_3: axis 0 0 1 -> -0 -0 -1; origin xyz=0.0514 0.0 0.0 rpy=0.0 0.0 0.0 -> xyz=0.0514 0 0 rpy=0 -0 0
