Commit message: gen: fix collision capsules being 43-57% too long
You were right to ask whether we were really using capsules. We were --
but the wrong size, which is worse than cylinders would have been.

Isaac Lab's replace_cylinders_with_capsules reads a URDF cylinder's `length`
as the capsule's CYLINDRICAL SECTION and adds a hemisphere of `radius` at
each end. The builder emitted the segment length directly, so every collision
shape came out 2r longer than its joint spacing:

    segment   joint spacing   collision capsule   error
    PP            47.00 mm         67.33 mm       +43%
    MP            31.50 mm         49.37 mm       +57%
    DP            26.01 mm         40.69 mm       +56%

Every capsule overhung both of its joints. Fingers were physically longer
than their kinematics claimed, and adjacent segments overlapped by
construction -- which is a large part of the self-collision I have been
chasing for the last several rounds. Some of those "overlaps" were an
artifact of this, not of the design space.

Fix: emit `length - 2r` for the COLLISION cylinder so the converted capsule
totals `length`. The VISUAL stays a full-length cylinder -- it is not
converted -- so both now span exactly the joint spacing. Verified in the
converted USD: PP collision is now height 26.67 + 2x10.17 = 47.00 mm.

Densities are refitted against the corrected volume, since they were
calibrated to weigh SHARPA's links at the inflated shape:

    mc  1073 -> 1854      pp  2105 -> 3169
    mp  2305 -> 3918      dp   678 -> 1149

These land much closer to the densities implied by the real mesh volumes
(pp 3032, mp 3131, dp 1644), which the over-long capsules did not -- an
independent sign the corrected shape is the better model.

cylinder_part() now lives in sharpa_anchors, shared by the URDF builder, the
degenerate-link path and the self-collision checker, so the shape the tools
assume cannot drift from the shape PhysX simulates.

Effect on self-collision at the home pose, same six sampled hands:
    before  14 pairs, 2/6 clean
    after    6 pairs, 4/6 clean
SHARPA and gen_sharpa_like are both clean. Masses still match SHARPA to
0.05% and kinematics to 0.002 mm; whole-hand mass 1203.7 -> 1212.6 g
(7.4% -> 6.7% light).

Co-Authored-By: Claude Opus 5 (1M context) <noreply@anthropic.com>

File: assets/urdf/generated/gen_0051_000.urdf (robot description, URDF)
Before this commit: robot iiwa14_gen_0051_000, 45 links, 44 joints
Links:
- link gen_f0_DP: mass 0.00359391344 -> 0.0043877249; geometry collision cylinder length=0.0235721264 radius=0.00618111626; visual cylinder length=0.0359343589 radius=0.00618111626
- link gen_f0_MP: mass 0.0155989878 -> 0.0160211741; geometry collision cylinder length=0.0129558426 radius=0.00752484254; visual cylinder length=0.0280055276 radius=0.00752484254
- link gen_f0_PP: mass 0.0299099273 -> 0.0325275627; geometry collision cylinder length=0.0331445315 radius=0.00856295734; visual cylinder length=0.0502704462 radius=0.00856295734
- link gen_f1_DP: mass 0.00575133083 -> 0.00637865051; geometry collision cylinder length=0.0190118697 radius=0.00775831711; visual cylinder length=0.0345285039 radius=0.00775831711
- link gen_f1_MP: mass 0.0331009845 -> 0.0355130659; geometry collision cylinder length=0.019752144 radius=0.0094449145; visual cylinder length=0.038641973 radius=0.0094449145
- link gen_f1_PP: mass 0.0429938942 -> 0.0400062521; geometry collision cylinder length=0.0204581184 radius=0.0107479192; visual cylinder length=0.0419539569 radius=0.0107479192
- link gen_f2_DP: mass 0.00197929227 -> 0.00235621117; geometry collision cylinder length=0.017497111 radius=0.00517271707; visual cylinder length=0.0278425451 radius=0.00517271707
- link gen_f2_MP: mass 0.0137486092 -> 0.0172178931; geometry collision cylinder length=0.0268814984 radius=0.00629722526; visual cylinder length=0.0394759489 radius=0.00629722526
- link gen_f2_PP: mass 0.023411404 -> 0.0279186427; geometry collision cylinder length=0.0450591049 radius=0.00716598001; visual cylinder length=0.0593910649 radius=0.00716598001

File: assets/urdf/generated/gen_0051_001.urdf (robot description, URDF)
Before this commit: robot iiwa14_gen_0051_001, 45 links, 44 joints
Links:
- link gen_f0_DP: mass 0.00167930764 -> 0.00197052855; geometry collision cylinder length=0.0156642248 radius=0.00495135121; visual cylinder length=0.0255669272 radius=0.00495135121
- link gen_f0_MC: mass 0.0354727986 -> 0.0353543201; geometry collision cylinder length=0.0182066195 radius=0.0130554364; visual cylinder length=0.0443174922 radius=0.0130554364
- link gen_f0_MP: mass 0.0110098886 -> 0.0133195056; geometry collision cylinder length=0.0217481526 radius=0.00602773619; visual cylinder length=0.033803625 radius=0.00602773619
- link gen_f0_PP: mass 0.0176015401 -> 0.020073001; geometry collision cylinder length=0.0337100834 radius=0.00685931268; visual cylinder length=0.0474287087 radius=0.00685931268
- link gen_f1_DP: mass 0.00571463418 -> 0.0063535851; geometry collision cylinder length=0.0191514104 radius=0.00772971916; visual cylinder length=0.0346108487 radius=0.00772971916
- link gen_f1_MP: mass 0.0246228118 -> 0.021333497; geometry collision cylinder length=0.00702782972 radius=0.00941009957; visual cylinder length=0.0258480289 radius=0.00941009957
- link gen_f1_PP: mass 0.0334662763 -> 0.0259350617; geometry collision cylinder length=0.00844208877 radius=0.0107083013; visual cylinder length=0.0298586914 radius=0.0107083013

File: assets/urdf/generated/gen_0051_002.urdf (robot description, URDF)
Before this commit: robot iiwa14_gen_0051_002, 45 links, 44 joints
Links:
- link gen_f0_DP: mass 0.00254156038 -> 0.00208726772; geometry collision cylinder length=0.00368533532 radius=0.0067510103; visual cylinder length=0.0171873559 radius=0.0067510103
- link gen_f0_MC: mass 0.112231004 -> 0.12816308; geometry collision cylinder length=0.0457121334 radius=0.0178006733; visual cylinder length=0.08131348 radius=0.0178006733
- link gen_f0_MP: mass 0.0206071099 -> 0.0213554208; geometry collision cylinder length=0.0147297845 radius=0.00821862707; visual cylinder length=0.0311670386 radius=0.00821862707
- link gen_f0_PP: mass 0.023818276 -> 0.0195704381; geometry collision cylinder length=0.010005495 radius=0.00935245524; visual cylinder length=0.0287104054 radius=0.00935245524
- link gen_f1_DP: mass 0.00143537349 -> 0.0013639563; geometry collision cylinder length=0.00644189816 radius=0.00529104414; visual cylinder length=0.0170239864 radius=0.00529104414
- link gen_f1_MC: mass 0.0582740973 -> 0.0690314526; geometry collision cylinder length=0.0422944514 radius=0.013951119; visual cylinder length=0.0701966895 radius=0.013951119
- link gen_f1_MP: mass 0.0104833914 -> 0.0112373201; geometry collision cylinder length=0.0134175207 radius=0.0064412757; visual cylinder length=0.0263000721 radius=0.0064412757
- link gen_f1_PP: mass 0.0140287945 -> 0.013279029; geometry collision cylinder length=0.0150540476 radius=0.00732990342; visual cylinder length=0.0297138545 radius=0.00732990342
- link gen_f2_DP: mass 0.0073193537 -> 0.00766433973; geometry collision cylinder length=0.0164989745 radius=0.00869380188; visual cylinder length=0.0338865783 radius=0.00869380188
- link gen_f2_MC: mass 0.132552848 -> 0.0935430428
- link gen_f2_MP: mass 0.0449129709 -> 0.0471434473; geometry collision cylinder length=0.0200831676 radius=0.0105837663; visual cylinder length=0.0412507003 radius=0.0105837663
- link gen_f2_PP: mass 0.0716708454 -> 0.0731149909; geometry collision cylinder length=0.0345742996 radius=0.0120438852; visual cylinder length=0.05866207 radius=0.0120438852
- link gen_f3_DP: mass 0.00118037698 -> 0.0011810698; geometry collision cylinder length=0.00749325627 radius=0.00484282576; visual cylinder length=0.0171789078 radius=0.00484282576
- link gen_f3_MP: mass 0.0108384487 -> 0.0133749307; geometry collision cylinder length=0.0234037683 radius=0.00589561816; visual cylinder length=0.0351950046 radius=0.00589561816
- link gen_f3_PP: mass 0.0175264599 -> 0.0203732919; geometry collision cylinder length=0.0365229999 radius=0.00670896786; visual cylinder length=0.0499409357 radius=0.00670896786

File: assets/urdf/generated/gen_0051_003.urdf (robot description, URDF)
Before this commit: robot iiwa14_gen_0051_003, 45 links, 44 joints
Links:
- link gen_f0_DP: mass 0.00281571893 -> 0.00324595053; geometry collision cylinder length=0.0173796247 radius=0.00595872628; visual cylinder length=0.0292970772 radius=0.00595872628
- link gen_f0_MP: mass 0.0147101229 -> 0.0156024336; geometry collision cylinder length=0.0144182788 radius=0.00725410672; visual cylinder length=0.0289264923 radius=0.00725410672
- link gen_f0_PP: mass 0.0249992179 -> 0.0264359836; geometry collision cylinder length=0.0279638011 radius=0.00825487126; visual cylinder length=0.0444735436 radius=0.00825487126
- link gen_f1_DP: mass 0.00370990937 -> 0.00372097868; geometry collision cylinder length=0.0110832724 radius=0.007085645; visual cylinder length=0.0252545624 radius=0.007085645
- link gen_f1_MP: mass 0.0202816017 -> 0.018667818; geometry collision cylinder length=0.00888285631 radius=0.00862600874; visual cylinder length=0.0261348738 radius=0.00862600874
- link gen_f1_PP: mass 0.0411664136 -> 0.0431435162; geometry collision cylinder length=0.0318901269 radius=0.00981603861; visual cylinder length=0.0515222041 radius=0.00981603861
- link gen_f2_DP: mass 0.00549600308 -> 0.00527570306; geometry collision cylinder length=0.0105274788 radius=0.00824158162; visual cylinder length=0.027010642 radius=0.00824158162
- link gen_f2_MP: mass 0.0321783122 -> 0.0298229883; geometry collision cylinder length=0.0106930636 radius=0.0100332369; visual cylinder length=0.0307595375 radius=0.0100332369
- link gen_f2_PP: mass 0.0623639909 -> 0.0642542643; geometry collision cylinder length=0.0342905554 radius=0.0114174057; visual cylinder length=0.0571253667 radius=0.0114174057
- link gen_f3_DP: mass 0.00440930274 -> 0.00367648317; geometry collision cylinder length=0.0048630828 radius=0.00807294619; visual cylinder length=0.0210089752 radius=0.00807294619
- link gen_f3_MP: mass 0.0383430586 -> 0.0417946711; geometry collision cylinder length=0.0220533945 radius=0.00982794147; visual cylinder length=0.0417092774 radius=0.00982794147
- link gen_f3_PP: mass 0.04338763 -> 0.0374679581; geometry collision cylinder length=0.0151795873 radius=0.011183788; visual cylinder length=0.0375471632 radius=0.011183788
- link gen_f4_DP: mass 0.00308022994 -> 0.002879475; geometry collision cylinder length=0.00773193213 radius=0.00687141858; visual cylinder length=0.0214747693 radius=0.00687141858
- link gen_f4_MC: mass 0.106406906 -> 0.114524079; geometry collision cylinder length=0.0357426335 radius=0.0181181589; visual cylinder length=0.0719789513 radius=0.0181181589
- link gen_f4_MP: mass 0.0225091582 -> 0.0238435356; geometry collision cylinder length=0.0165308902 radius=0.00836521118; visual cylinder length=0.0332613126 radius=0.00836521118
- link gen_f4_PP: mass 0.0293688723 -> 0.0270395794; geometry collision cylinder length=0.0172821702 radius=0.00951926185; visual cylinder length=0.0363206939 radius=0.00951926185

File: assets/urdf/generated/gen_0051_004.urdf (robot description, URDF)
Before this commit: robot iiwa14_gen_0051_004, 45 links, 44 joints
Links:
- link gen_f0_DP: mass 0.00509454517 -> 0.00499246251; geometry collision cylinder length=0.0111992857 radius=0.00796212543; visual cylinder length=0.0271235366 radius=0.00796212543
- link gen_f0_MP: mass 0.0220447851 -> 0.0150460215; geometry collision cylinder length=8.73174129e-05 radius=0.00969302915; visual cylinder length=0.0194733757 radius=0.00969302915
- link gen_f0_PP: mass 0.0590543234 -> 0.0621849819; geometry collision cylinder length=0.0366349591 radius=0.0110302634; visual cylinder length=0.0586954859 radius=0.0110302634
- link gen_f1_DP: mass 0.00395655615 -> 0.00474582561; geometry collision cylinder length=0.0227029027 radius=0.00647691904; visual cylinder length=0.0356567408 radius=0.00647691904
- link gen_f1_MC: mass 0.0431046071 -> 0.0386801084
- link gen_f1_MP: mass 0.0243477585 -> 0.0293101279; geometry collision cylinder length=0.0277903418 radius=0.00788495052; visual cylinder length=0.0435602428 radius=0.00788495052
- link gen_f1_PP: mass 0.0264087973 -> 0.0253747283; geometry collision cylinder length=0.0196962419 radius=0.00897274523; visual cylinder length=0.0376417323 radius=0.00897274523
- link gen_f2_DP: mass 0.00234720216 -> 0.00283709715; geometry collision cylinder length=0.0196587143 radius=0.00540827796; visual cylinder length=0.0304752702 radius=0.00540827796
- link gen_f2_MC: mass 0.0668262344 -> 0.0816548167; geometry collision cylinder length=0.0499289958 radius=0.0142602344; visual cylinder length=0.0784494645 radius=0.0142602344
- link gen_f2_MP: mass 0.0147869533 -> 0.0181038881; geometry collision cylinder length=0.0251535985 radius=0.00658399524; visual cylinder length=0.038321589 radius=0.00658399524
- link gen_f2_PP: mass 0.0198120058 -> 0.0214526536; geometry collision cylinder length=0.0283993667 radius=0.00749231231; visual cylinder length=0.0433839913 radius=0.00749231231
- link gen_f3_DP: mass 0.00252261914 -> 0.00294817975; geometry collision cylinder length=0.0176624806 radius=0.00568766632; visual cylinder length=0.0290378132 radius=0.00568766632
- link gen_f3_MP: mass 0.0177103572 -> 0.021925994; geometry collision cylinder length=0.0279256395 radius=0.00692412044; visual cylinder length=0.0417738803 radius=0.00692412044
- link gen_f3_PP: mass 0.0203858364 -> 0.0209505983; geometry collision cylinder length=0.0233921265 radius=0.00787936062; visual cylinder length=0.0391508477 radius=0.00787936062
- link gen_f4_DP: mass 0.00665406621 -> 0.00637464914; geometry collision cylinder length=0.0111250815 radius=0.00879155676; visual cylinder length=0.028708195 radius=0.00879155676
- link gen_f4_MP: mass 0.0396001721 -> 0.0371191797; geometry collision cylinder length=0.012058113 radius=0.0107027724; visual cylinder length=0.0334636577 radius=0.0107027724
- link gen_f4_PP: mass 0.0662185803 -> 0.0637201949; geometry collision cylinder length=0.0269118981 radius=0.0121793091; visual cylinder length=0.0512705163 radius=0.0121793091

File: assets/urdf/generated/gen_0051_005.urdf (robot description, URDF)
Before this commit: robot iiwa14_gen_0051_005, 45 links, 44 joints
Links:
- link gen_f0_DP: mass 0.00467296247 -> 0.00534708514; geometry collision cylinder length=0.0199973989 radius=0.00709166003; visual cylinder length=0.034180719 radius=0.00709166003
- link gen_f0_MC: mass 0.123233915 -> 0.136713144; geometry collision cylinder length=0.042201551 radius=0.0186988788; visual cylinder length=0.0795993086 radius=0.0186988788
- link gen_f0_MP: mass 0.0248385084 -> 0.0263716968; geometry collision cylinder length=0.0172364641 radius=0.00863333139; visual cylinder length=0.0345031269 radius=0.00863333139
- link gen_f0_PP: mass 0.0383983308 -> 0.038928252; geometry collision cylinder length=0.027415684 radius=0.00982437148; visual cylinder length=0.047064427 radius=0.00982437148
- link gen_f1_DP: mass 0.00495874145 -> 0.00466576844; geometry collision cylinder length=0.0093268398 radius=0.00803176984; visual cylinder length=0.0253903795 radius=0.00803176984
- link gen_f1_MP: mass 0.0289822329 -> 0.0262423194; geometry collision cylinder length=0.00926464894 radius=0.00977781371; visual cylinder length=0.0288202764 radius=0.00977781371
- link gen_f1_PP: mass 0.0399756385 -> 0.0327552995; geometry collision cylinder length=0.0117412311 radius=0.0111267447; visual cylinder length=0.0339947205 radius=0.0111267447

File: assets/urdf/generated/gen_sharpa_like.urdf (robot description, URDF)
Before this commit: robot iiwa14_gen_sharpa_like, 45 links, 44 joints
Links:
- link gen_f0_DP: mass 0.00428760247 -> 0.00441595447; geometry collision cylinder length=0.0129338764 radius=0.00733806181; visual cylinder length=0.02761 radius=0.00733806181
- link gen_f0_MC: mass 0.115997537 -> 0.115995746; geometry collision cylinder length=0.0274008956 radius=0.0193485768; visual cylinder length=0.0660980491 radius=0.0193485768
- link gen_f0_PP: mass 0.0359131707 -> 0.0331498526; geometry collision cylinder length=0.0186685558 radius=0.0101657221; visual cylinder length=0.039 radius=0.0101657221
- link gen_f1_DP: mass 0.0041041466 -> 0.00410494382; geometry collision cylinder length=0.0113338764 radius=0.00733806181; visual cylinder length=0.02601 radius=0.00733806181
- link gen_f1_MP: geometry collision cylinder length=0.013633402 radius=0.00893329899; visual cylinder length=0.0315 radius=0.00893329899
- link gen_f1_PP: geometry collision cylinder length=0.0266685558 radius=0.0101657221; visual cylinder length=0.047 radius=0.0101657221
- link gen_f2_DP: mass 0.0041041466 -> 0.00410494382; geometry collision cylinder length=0.0113338764 radius=0.00733806181; visual cylinder length=0.02601 radius=0.00733806181
- link gen_f2_MP: geometry collision cylinder length=0.013633402 radius=0.00893329899; visual cylinder length=0.0315 radius=0.00893329899
- link gen_f2_PP: geometry collision cylinder length=0.0266685558 radius=0.0101657221; visual cylinder length=0.047 radius=0.0101657221
- link gen_f3_DP: mass 0.0041041466 -> 0.00410494382; geometry collision cylinder length=0.0113338764 radius=0.00733806181; visual cylinder length=0.02601 radius=0.00733806181
- link gen_f3_MP: geometry collision cylinder length=0.013633402 radius=0.00893329899; visual cylinder length=0.0315 radius=0.00893329899
- link gen_f3_PP: geometry collision cylinder length=0.0266685558 radius=0.0101657221; visual cylinder length=0.047 radius=0.0101657221
- link gen_f4_DP: mass 0.0041041466 -> 0.00410494382; geometry collision cylinder length=0.0113338764 radius=0.00733806181; visual cylinder length=0.02601 radius=0.00733806181
- link gen_f4_MC: mass 0.0447323695 -> 0.0562504982
- link gen_f4_MP: geometry collision cylinder length=0.013633402 radius=0.00893329899; visual cylinder length=0.0315 radius=0.00893329899
- link gen_f4_PP: geometry collision cylinder length=0.0266685558 radius=0.0101657221; visual cylinder length=0.047 radius=0.0101657221

File: assets/urdf/generated/sharpa_like.urdf (robot description, URDF)
Before this commit: robot iiwa14_sharpa_like, 45 links, 44 joints
Links:
- link gen_f0_DP: mass 0.00428760247 -> 0.00441595447; geometry collision cylinder length=0.0129338764 radius=0.00733806181; visual cylinder length=0.02761 radius=0.00733806181
- link gen_f0_MC: mass 0.115997537 -> 0.115995746; geometry collision cylinder length=0.0274008956 radius=0.0193485768; visual cylinder length=0.0660980491 radius=0.0193485768
- link gen_f0_PP: mass 0.0359131707 -> 0.0331498526; geometry collision cylinder length=0.0186685558 radius=0.0101657221; visual cylinder length=0.039 radius=0.0101657221
- link gen_f1_DP: mass 0.0041041466 -> 0.00410494382; geometry collision cylinder length=0.0113338764 radius=0.00733806181; visual cylinder length=0.02601 radius=0.00733806181
- link gen_f1_MP: geometry collision cylinder length=0.013633402 radius=0.00893329899; visual cylinder length=0.0315 radius=0.00893329899
- link gen_f1_PP: geometry collision cylinder length=0.0266685558 radius=0.0101657221; visual cylinder length=0.047 radius=0.0101657221
- link gen_f2_DP: mass 0.0041041466 -> 0.00410494382; geometry collision cylinder length=0.0113338764 radius=0.00733806181; visual cylinder length=0.02601 radius=0.00733806181
- link gen_f2_MP: geometry collision cylinder length=0.013633402 radius=0.00893329899; visual cylinder length=0.0315 radius=0.00893329899
- link gen_f2_PP: geometry collision cylinder length=0.0266685558 radius=0.0101657221; visual cylinder length=0.047 radius=0.0101657221
- link gen_f3_DP: mass 0.0041041466 -> 0.00410494382; geometry collision cylinder length=0.0113338764 radius=0.00733806181; visual cylinder length=0.02601 radius=0.00733806181
- link gen_f3_MP: geometry collision cylinder length=0.013633402 radius=0.00893329899; visual cylinder length=0.0315 radius=0.00893329899
- link gen_f3_PP: geometry collision cylinder length=0.0266685558 radius=0.0101657221; visual cylinder length=0.047 radius=0.0101657221
- link gen_f4_DP: mass 0.0041041466 -> 0.00410494382; geometry collision cylinder length=0.0113338764 radius=0.00733806181; visual cylinder length=0.02601 radius=0.00733806181
- link gen_f4_MC: mass 0.0447323695 -> 0.0562504982
- link gen_f4_MP: geometry collision cylinder length=0.013633402 radius=0.00893329899; visual cylinder length=0.0315 radius=0.00893329899
- link gen_f4_PP: geometry collision cylinder length=0.0266685558 radius=0.0101657221; visual cylinder length=0.047 radius=0.0101657221
