Commit message: gen: capsule visuals, and a collision/visual toggle in the viewer
Visual geometry is now the same capsule as collision

    URDF has no capsule primitive and replace_cylinders_with_capsules only
    converts COLLISION geometry, so a generated finger rendered as a
    flat-ended cylinder while the thing being simulated had round ends.

    Each phalanx now emits its visual as a cylinder plus a sphere at both ends
    of the cylindrical section, which reproduces the collision capsule
    exactly. For a 47.00 mm phalanx of radius 10.17 mm: cylinder 26.67 mm
    centred at 23.50, spheres at 10.17 and 36.83 -- spanning 0 to 47.00, the
    joint spacing. Renders and videos now show the hand that is actually in
    contact with the object.

Viewer: "show geometry" toggle, collision | visual

    link_collision_meshes generalises to link_geometry_meshes(..., which=),
    with the old name kept as a thin alias since physics is always collision.

    The toggle changes only what is DRAWN. The self-collision check always
    runs on collision geometry whatever is on screen, because that is what
    PhysX resolves. Both arm mesh sets load once at startup and swap
    visibility rather than reloading.

    This also makes the two representations comparable by eye: they are the
    same capsule built two ways, so a visible mismatch means the builder has
    drifted.

Co-Authored-By: Claude Opus 5 (1M context) <noreply@anthropic.com>

File: assets/urdf/generated/gen_sharpa_like.urdf (robot description, URDF)
Before this commit: robot iiwa14_gen_sharpa_like, 45 links, 44 joints
Links:
- link gen_f0_DP: geometry collision cylinder length=0.0129338764 radius=0.00733806181; visual cylinder length=0.0129338764 radius=0.00733806181
- link gen_f0_MC: geometry collision cylinder length=0.0274008956 radius=0.0193485768; visual cylinder length=0.0274008956 radius=0.0193485768
- link gen_f0_PP: geometry collision cylinder length=0.0186685558 radius=0.0101657221; visual cylinder length=0.0186685558 radius=0.0101657221
- link gen_f1_DP: geometry collision cylinder length=0.0113338764 radius=0.00733806181; visual cylinder length=0.0113338764 radius=0.00733806181
- link gen_f1_MP: geometry collision cylinder length=0.013633402 radius=0.00893329899; visual cylinder length=0.013633402 radius=0.00893329899
- link gen_f1_PP: geometry collision cylinder length=0.0266685558 radius=0.0101657221; visual cylinder length=0.0266685558 radius=0.0101657221
- link gen_f2_DP: geometry collision cylinder length=0.0113338764 radius=0.00733806181; visual cylinder length=0.0113338764 radius=0.00733806181
- link gen_f2_MP: geometry collision cylinder length=0.013633402 radius=0.00893329899; visual cylinder length=0.013633402 radius=0.00893329899
- link gen_f2_PP: geometry collision cylinder length=0.0266685558 radius=0.0101657221; visual cylinder length=0.0266685558 radius=0.0101657221
- link gen_f3_DP: geometry collision cylinder length=0.0113338764 radius=0.00733806181; visual cylinder length=0.0113338764 radius=0.00733806181
- link gen_f3_MP: geometry collision cylinder length=0.013633402 radius=0.00893329899; visual cylinder length=0.013633402 radius=0.00893329899
- link gen_f3_PP: geometry collision cylinder length=0.0266685558 radius=0.0101657221; visual cylinder length=0.0266685558 radius=0.0101657221
- link gen_f4_DP: geometry collision cylinder length=0.0113338764 radius=0.00733806181; visual cylinder length=0.0113338764 radius=0.00733806181
- link gen_f4_MP: geometry collision cylinder length=0.013633402 radius=0.00893329899; visual cylinder length=0.013633402 radius=0.00893329899
- link gen_f4_PP: geometry collision cylinder length=0.0266685558 radius=0.0101657221; visual cylinder length=0.0266685558 radius=0.0101657221

File: assets/urdf/generated/sharpa_like.urdf (robot description, URDF)
Before this commit: robot iiwa14_sharpa_like, 45 links, 44 joints
Links:
- link gen_f0_DP: geometry collision cylinder length=0.0129338764 radius=0.00733806181; visual cylinder length=0.0129338764 radius=0.00733806181
- link gen_f0_MC: geometry collision cylinder length=0.0274008956 radius=0.0193485768; visual cylinder length=0.0274008956 radius=0.0193485768
- link gen_f0_PP: geometry collision cylinder length=0.0186685558 radius=0.0101657221; visual cylinder length=0.0186685558 radius=0.0101657221
- link gen_f1_DP: geometry collision cylinder length=0.0113338764 radius=0.00733806181; visual cylinder length=0.0113338764 radius=0.00733806181
- link gen_f1_MP: geometry collision cylinder length=0.013633402 radius=0.00893329899; visual cylinder length=0.013633402 radius=0.00893329899
- link gen_f1_PP: geometry collision cylinder length=0.0266685558 radius=0.0101657221; visual cylinder length=0.0266685558 radius=0.0101657221
- link gen_f2_DP: geometry collision cylinder length=0.0113338764 radius=0.00733806181; visual cylinder length=0.0113338764 radius=0.00733806181
- link gen_f2_MP: geometry collision cylinder length=0.013633402 radius=0.00893329899; visual cylinder length=0.013633402 radius=0.00893329899
- link gen_f2_PP: geometry collision cylinder length=0.0266685558 radius=0.0101657221; visual cylinder length=0.0266685558 radius=0.0101657221
- link gen_f3_DP: geometry collision cylinder length=0.0113338764 radius=0.00733806181; visual cylinder length=0.0113338764 radius=0.00733806181
- link gen_f3_MP: geometry collision cylinder length=0.013633402 radius=0.00893329899; visual cylinder length=0.013633402 radius=0.00893329899
- link gen_f3_PP: geometry collision cylinder length=0.0266685558 radius=0.0101657221; visual cylinder length=0.0266685558 radius=0.0101657221
- link gen_f4_DP: geometry collision cylinder length=0.0113338764 radius=0.00733806181; visual cylinder length=0.0113338764 radius=0.00733806181
- link gen_f4_MP: geometry collision cylinder length=0.013633402 radius=0.00893329899; visual cylinder length=0.013633402 radius=0.00893329899
- link gen_f4_PP: geometry collision cylinder length=0.0266685558 radius=0.0101657221; visual cylinder length=0.0266685558 radius=0.0101657221

Commit message: gen: ghosted joints were not actually locked — hold them with the actuator
A real physics bug, found because the wandb viewer disagreed with viser about
finger-object penetration. The viewer was right and the robot was wrong.

Ghosted joints were locked to [0, 1e-8] and given a deliberately weak actuator
(stiffness 0.01, effort 1e-3), on the theory that the limit does the holding.
PhysX joint limits are COMPLIANT, not rigid constraints. Under grasp forces the
"locked" joints were pushed straight open: in the training capture at step
360599, gen_f3_CMC_FE reached -0.364 rad (21 deg) against limits of [0, 0],
with 4832 limit violations across 600 frames.

That made a ghosted finger move, so the design space's premise -- that only
ACTIVE joints matter and ghosted ones are inert padding -- was false for every
generated hand.

It surfaced as apparent interpenetration because urdf-loader CLAMPS joint
values to URDF limits while the physics did not, so the browser drew that
finger 21 deg from where the simulator had it. SHARPA and Allegro were
unaffected because they have no ghosted joints, which is exactly why only the
generated runs looked wrong.

Fix: hold ghost joints with the actuator instead of the limit. Stiffness and
damping are 10x the strongest live tier, armature is the largest, and the
effort limit is the slot's real value rather than throttled to 1e-3. Cost is
solver work on joints that never move -- the price of a fixed-shape
articulation.

Verified under load (new --check ghost_load, Isaac Sim): driving every joint to
both extremes for 240 steps, the worst ghosted joint now moves 0.060 mrad,
against 364 mrad before. That check is the one that was missing when ghosting
landed; it would have caught this the same day.

Co-Authored-By: Claude Opus 5 (1M context) <noreply@anthropic.com>

File: assets/urdf/generated/gen_sharpa_like.urdf (robot description, URDF)
Before this commit: robot iiwa14_gen_sharpa_like, 45 links, 44 joints
Joints:
- joint gen_f0_PIP: limit lower=0 upper=1e-08 effort=0.001 velocity=11.618316 -> lower=0 upper=1e-08 effort=0.638 velocity=11.618316
- joint gen_f1_CMC_AA: limit lower=0 upper=1e-08 effort=0.001 velocity=11.8407683 -> lower=0 upper=1e-08 effort=3.3 velocity=11.8407683
- joint gen_f1_CMC_FE: limit lower=0 upper=1e-08 effort=0.001 velocity=11.8407683 -> lower=0 upper=1e-08 effort=3.3 velocity=11.8407683
- joint gen_f2_CMC_AA: limit lower=0 upper=1e-08 effort=0.001 velocity=11.8407683 -> lower=0 upper=1e-08 effort=3.3 velocity=11.8407683
- joint gen_f2_CMC_FE: limit lower=0 upper=1e-08 effort=0.001 velocity=11.8407683 -> lower=0 upper=1e-08 effort=3.3 velocity=11.8407683
- joint gen_f3_CMC_AA: limit lower=0 upper=1e-08 effort=0.001 velocity=11.8407683 -> lower=0 upper=1e-08 effort=3.3 velocity=11.8407683
- joint gen_f3_CMC_FE: limit lower=0 upper=1e-08 effort=0.001 velocity=11.8407683 -> lower=0 upper=1e-08 effort=3.3 velocity=11.8407683
- joint gen_f4_CMC_AA: limit lower=0 upper=1e-08 effort=0.001 velocity=11.8407683 -> lower=0 upper=1e-08 effort=3.3 velocity=11.8407683
