Commit message: Ten hands: USD-safe names in onboarding; all 7 left hands pass smoke; training submitted
Co-Authored-By: Claude Opus 5.5 <noreply@anthropic.com>
Claude-Session: https://claude.ai/code/session_01VEjfLD7vkNCwPYPC2HsL71

File: assets/urdf/unified_commercial_hands/allegro/allegro_left.urdf (robot description, URDF)
Before this commit: robot allegro_left, 23 links, 22 joints
Links:
- removed link link_0.0
- removed link link_1.0
- removed link link_10.0
- removed link link_11.0
- removed link link_11.0_tip
- removed link link_12.0
- removed link link_13.0
- removed link link_14.0
- removed link link_15.0
- removed link link_15.0_tip
- removed link link_2.0
- removed link link_3.0
- removed link link_3.0_tip
- removed link link_4.0
- removed link link_5.0
- removed link link_6.0
- removed link link_7.0
- removed link link_7.0_tip
- removed link link_8.0
- removed link link_9.0
- added link link_0_0, mass 0.0119; collision box size=0.0196 0.0275 0.0164; visual mesh filename=vendor_left/meshes/link_0.0.obj
- added link link_10_0, mass 0.0355; collision box size=0.0196 0.0275 0.0384; visual mesh filename=vendor_left/meshes/link_2.0.obj
- added link link_11_0, mass 0.0096; collision box size=0.0196 0.0269 0.022; visual mesh filename=vendor_left/meshes/link_3.0.obj
- added link link_11_0_tip, mass 0.0168; collision mesh filename=vendor_left/meshes/collision_link_tip.obj; visual mesh filename=vendor_left/meshes/link_tip.obj
- added link link_12_0, mass 0.0176; collision box size=0.0358 0.034 0.0455; visual mesh filename=vendor_left/meshes/link_12.0_left.obj
- added link link_13_0, mass 0.0119; collision box size=0.0196 0.0275 0.0177; visual mesh filename=vendor_left/meshes/link_13.0.obj
- added link link_14_0, mass 0.038; collision box size=0.0196 0.0275 0.0514; visual mesh filename=vendor_left/meshes/link_14.0.obj
- added link link_15_0, mass 0.0388; collision box size=0.0196 0.0269 0.04; visual mesh filename=vendor_left/meshes/link_15.0.obj
- added link link_15_0_tip, mass 0.0168; collision mesh filename=vendor_left/meshes/collision_link_tip.obj; visual mesh filename=vendor_left/meshes/link_tip.obj
- added link link_1_0, mass 0.065; collision box size=0.0196 0.0275 0.054; visual mesh filename=vendor_left/meshes/link_1.0.obj
- added link link_2_0, mass 0.0355; collision box size=0.0196 0.0275 0.0384; visual mesh filename=vendor_left/meshes/link_2.0.obj
- added link link_3_0, mass 0.02; collision box size=0.0196 0.0269 0.022; visual mesh filename=vendor_left/meshes/link_3.0.obj
- added link link_3_0_tip, mass 0.0168; collision mesh filename=vendor_left/meshes/collision_link_tip.obj; visual mesh filename=vendor_left/meshes/link_tip.obj
- added link link_4_0, mass 0.005; collision box size=0.0196 0.0275 0.0164; visual mesh filename=vendor_left/meshes/link_0.0.obj
- added link link_5_0, mass 0.065; collision box size=0.0196 0.0275 0.054; visual mesh filename=vendor_left/meshes/link_1.0.obj
- added link link_6_0, mass 0.0355; collision box size=0.0196 0.0275 0.0384; visual mesh filename=vendor_left/meshes/link_2.0.obj
- added link link_7_0, mass 0.0388; collision box size=0.0196 0.0269 0.022; visual mesh filename=vendor_left/meshes/link_3.0.obj
- added link link_7_0_tip, mass 0.0096; collision mesh filename=vendor_left/meshes/collision_link_tip.obj; visual mesh filename=vendor_left/meshes/link_tip.obj
- added link link_8_0, mass 0.005; collision box size=0.0196 0.0275 0.0164; visual mesh filename=vendor_left/meshes/link_0.0.obj
- added link link_9_0, mass 0.065; collision box size=0.0196 0.0275 0.054; visual mesh filename=vendor_left/meshes/link_1.0.obj
Joints:
- removed joint joint_0.0
- removed joint joint_1.0
- removed joint joint_10.0
- removed joint joint_11.0
- removed joint joint_11.0_tip
- removed joint joint_12.0
- removed joint joint_13.0
- removed joint joint_14.0
- removed joint joint_15.0
- removed joint joint_15.0_tip
- removed joint joint_2.0
- removed joint joint_3.0
- removed joint joint_3.0_tip
- removed joint joint_4.0
- removed joint joint_5.0
- removed joint joint_6.0
- removed joint joint_7.0
- removed joint joint_7.0_tip
- removed joint joint_8.0
- removed joint joint_9.0
- added joint joint_0_0: type revolute, parent base_link, child link_0_0, origin xyz=0 0.0435 -0.001542 rpy=-0.08726646255 0 0, axis 0 0 1, limit lower=-0.47 upper=0.47 effort=10 velocity=3.14
- added joint joint_10_0: type revolute, parent link_9_0, child link_10_0, origin xyz=0 0 0.054, axis 0 1 0, limit lower=-0.174 upper=1.709 effort=10 velocity=3.14
- added joint joint_11_0: type revolute, parent link_10_0, child link_11_0, origin xyz=0 0 0.0384, axis 0 1 0, limit lower=-0.227 upper=1.618 effort=10 velocity=3.14
- added joint joint_11_0_tip: type fixed, parent link_11_0, child link_11_0_tip, origin xyz=0 0 0.0387 rpy=0 0 0
- added joint joint_12_0: type revolute, parent base_link, child link_12_0, origin xyz=-0.0182 -0.019333 -0.045987 rpy=0 -1.65806278845 1.5707963259, axis 1 0 0, limit lower=0.263 upper=1.396 effort=10 velocity=3.14
- added joint joint_13_0: type revolute, parent link_12_0, child link_13_0, origin xyz=-0.027 0.005 0.0399, axis 0 0 -1, limit lower=-0.105 upper=1.163 effort=10 velocity=3.14
- added joint joint_14_0: type revolute, parent link_13_0, child link_14_0, origin xyz=0 0 0.0177, axis 0 1 0, limit lower=-0.189 upper=1.644 effort=10 velocity=3.14
- added joint joint_15_0: type revolute, parent link_14_0, child link_15_0, origin xyz=0 0 0.0514, axis 0 1 0, limit lower=-0.162 upper=1.719 effort=10 velocity=3.14
- added joint joint_15_0_tip: type fixed, parent link_15_0, child link_15_0_tip, origin xyz=0 0 0.0543 rpy=0 0 0
- added joint joint_1_0: type revolute, parent link_0_0, child link_1_0, origin xyz=0 0 0.0164, axis 0 1 0, limit lower=-0.196 upper=1.61 effort=10 velocity=3.14
- added joint joint_2_0: type revolute, parent link_1_0, child link_2_0, origin xyz=0 0 0.054, axis 0 1 0, limit lower=-0.174 upper=1.709 effort=10 velocity=3.14
- added joint joint_3_0: type revolute, parent link_2_0, child link_3_0, origin xyz=0 0 0.0384, axis 0 1 0, limit lower=-0.227 upper=1.618 effort=10 velocity=3.14
- added joint joint_3_0_tip: type fixed, parent link_3_0, child link_3_0_tip, origin xyz=0 0 0.0387 rpy=0 0 0
- added joint joint_4_0: type revolute, parent base_link, child link_4_0, origin xyz=0 0 0.0007 rpy=0.0 0 0, axis 0 0 1, limit lower=-0.47 upper=0.47 effort=10 velocity=3.14
- added joint joint_5_0: type revolute, parent link_4_0, child link_5_0, origin xyz=0 0 0.0164, axis 0 1 0, limit lower=-0.196 upper=1.61 effort=10 velocity=3.14
- added joint joint_6_0: type revolute, parent link_5_0, child link_6_0, origin xyz=0 0 0.054, axis 0 1 0, limit lower=-0.174 upper=1.709 effort=10 velocity=3.14
- added joint joint_7_0: type revolute, parent link_6_0, child link_7_0, origin xyz=0 0 0.0384, axis 0 1 0, limit lower=-0.227 upper=1.618 effort=10 velocity=3.14
- added joint joint_7_0_tip: type fixed, parent link_7_0, child link_7_0_tip, origin xyz=0 0 0.0387 rpy=0 0 0
- added joint joint_8_0: type revolute, parent base_link, child link_8_0, origin xyz=0 -0.0435 -0.001542 rpy=0.08726646255 0 0, axis 0 0 1, limit lower=-0.47 upper=0.47 effort=10 velocity=3.14
- added joint joint_9_0: type revolute, parent link_8_0, child link_9_0, origin xyz=0 0 0.0164, axis 0 1 0, limit lower=-0.196 upper=1.61 effort=10 velocity=3.14

File: assets/urdf/unified_commercial_hands/leap/leap_left.urdf (robot description, URDF)
Before this commit: robot leap_left, 21 links, 20 joints
Joints:
- removed joint 0
- removed joint 1
- removed joint 10
- removed joint 11
- removed joint 12
- removed joint 13
- removed joint 14
- removed joint 15
- removed joint 2
- removed joint 3
- removed joint 4
- removed joint 5
- removed joint 6
- removed joint 7
- removed joint 8
- removed joint 9
- added joint j0: type revolute, parent mcp_joint, child pip, origin xyz=-0.0122 0.03810 0.01450 rpy=-1.57079 0 1.57079, axis 0 0 -1, limit lower=-1.047 upper=1.047 effort=0.95 velocity=8.48
- added joint j1: type revolute, parent palm_lower_left, child mcp_joint, origin xyz=-0.0825 -0.0857 0.0078 rpy=1.57079 1.57079 0, axis 0 0 -1, limit lower=-0.314 upper=2.23 effort=0.95 velocity=8.48
- added joint j10: type revolute, parent pip_3, child dip_3, origin xyz=0.015 0.0143 -0.013 rpy=1.57079 -1.57079 0, axis 0 0 -1, limit lower=-0.506 upper=1.885 effort=0.95 velocity=8.48
- added joint j11: type revolute, parent dip_3, child fingertip_3, origin xyz=0 -0.03609 0.0002 rpy=0 0 0, axis 0 0 -1, limit lower=-0.366 upper=2.042 effort=0.95 velocity=8.48
- added joint j12: type revolute, parent palm_lower_left, child thumb_left_temp_base, origin xyz=-0.1448 -0.0900 0.0049 rpy=0 1.57079 0, axis 0 0 -1, limit lower=-2.094 upper=0.349 effort=0.95 velocity=8.48
- added joint j13: type revolute, parent thumb_left_temp_base, child thumb_pip, origin xyz=0 -0.0143 -0.013 rpy=-1.57079 -1.57079 0, axis 0 0 -1, limit lower=-2.443 upper=0.47 effort=0.95 velocity=8.48
- added joint j14: type revolute, parent thumb_pip, child thumb_dip, origin xyz=0 0.0145 -0.017 rpy=-1.57079 0 0, axis 0 0 -1, limit lower=-1.20 upper=1.90 effort=0.95 velocity=8.48
- added joint j15: type revolute, parent thumb_dip, child thumb_fingertip, origin xyz=0 0.0466 0.0002 rpy=0 0 3.14159, axis 0 0 -1, limit lower=-1.34 upper=1.88 effort=0.95 velocity=8.48
- added joint j2: type revolute, parent pip, child dip, origin xyz=0.015 0.0143 -0.013 rpy=1.57079 -1.57079 0, axis 0 0 -1, limit lower=-0.506 upper=1.885 effort=0.95 velocity=8.48
- added joint j3: type revolute, parent dip, child fingertip, origin xyz=0 -0.0361 0.0002 rpy=0 0 0, axis 0 0 -1, limit lower=-0.366 upper=2.042 effort=0.95 velocity=8.48
- added joint j4: type revolute, parent mcp_joint_2, child pip_2, origin xyz=-0.0122 0.0381 0.0145 rpy=-1.57079 0 1.57079, axis 0 0 -1, limit lower=-1.047 upper=1.047 effort=0.95 velocity=8.48
- added joint j5: type revolute, parent palm_lower_left, child mcp_joint_2, origin xyz=-0.0825 -0.0403 0.0078 rpy=1.57079 1.57079 0, axis 0 0 -1, limit lower=-0.314 upper=2.23 effort=0.95 velocity=8.48
- added joint j6: type revolute, parent pip_2, child dip_2, origin xyz=0.015 0.0143 -0.013 rpy=1.57079 -1.57079 0, axis 0 0 -1, limit lower=-0.506 upper=1.885 effort=0.95 velocity=8.48
- added joint j7: type revolute, parent dip_2, child fingertip_2, origin xyz=0 -0.0361 0.0002 rpy=0 0 0, axis 0 0 -1, limit lower=-0.366 upper=2.042 effort=0.95 velocity=8.48
- added joint j8: type revolute, parent mcp_joint_3, child pip_3, origin xyz=-0.0122 0.0381 0.0145 rpy=-1.57079 0 1.57079, axis 0 0 -1, limit lower=-1.047 upper=1.047 effort=0.95 velocity=8.48
- added joint j9: type revolute, parent palm_lower_left, child mcp_joint_3, origin xyz=-0.0825 0.0051 0.0078 rpy=1.57079 1.57079 0, axis 0 0 -1, limit lower=-0.314 upper=2.23 effort=0.95 velocity=8.48
