Commit message: Tesollo: STL copies of the Collada visual meshes for the wandb viewer
The viewer loads STL/OBJ/glTF only, so the left Tesollo rendered empty.
onboard.py now converts .dae visuals to <hand>/visual_stl/*.stl (same
frame and scale: bounds match the collision meshes exactly). Collision,
spec and report are unchanged.

Co-Authored-By: Claude Opus 5.5 (1M context) <noreply@anthropic.com>
Claude-Session: https://claude.ai/code/session_01VEjfLD7vkNCwPYPC2HsL71

File: assets/urdf/unified_commercial_hands/tesollo/tesollo_left.urdf (robot description, URDF)
Before this commit: robot dg5f_left, 26 links, 25 joints
Links:
- link ll_dg_1_1: geometry collision mesh filename=vendor_left/meshes/ll_dg_1_1_c.STL; visual mesh filename=visual_stl/ll_dg_1_1.stl
- link ll_dg_1_2: geometry collision mesh filename=vendor_left/meshes/ll_dg_1_2_c.STL; visual mesh filename=visual_stl/ll_dg_1_2.stl
- link ll_dg_1_3: geometry collision mesh filename=vendor_left/meshes/ll_dg_1_3_c.STL; visual mesh filename=visual_stl/ll_dg_1_3.stl
- link ll_dg_1_4: geometry collision mesh filename=vendor_left/meshes/ll_dg_1_4_c.STL; visual mesh filename=visual_stl/ll_dg_1_4.stl
- link ll_dg_1_tip: geometry collision mesh filename=vendor_left/meshes/ll_dg_1_tip_c.STL; visual mesh filename=visual_stl/ll_dg_1_tip.stl
- link ll_dg_2_1: geometry collision mesh filename=vendor_left/meshes/ll_dg_2_1_c.STL; visual mesh filename=visual_stl/ll_dg_2_1.stl
- link ll_dg_2_2: geometry collision mesh filename=vendor_left/meshes/ll_dg_2_2_c.STL; visual mesh filename=visual_stl/ll_dg_2_2.stl
- link ll_dg_2_3: geometry collision mesh filename=vendor_left/meshes/ll_dg_2_3_c.STL; visual mesh filename=visual_stl/ll_dg_2_3.stl
- link ll_dg_2_4: geometry collision mesh filename=vendor_left/meshes/ll_dg_2_4_c.STL; visual mesh filename=visual_stl/ll_dg_2_4.stl
- link ll_dg_2_tip: geometry collision mesh filename=vendor_left/meshes/ll_dg_2_tip_c.STL; visual mesh filename=visual_stl/ll_dg_2_tip.stl
- link ll_dg_3_1: geometry collision mesh filename=vendor_left/meshes/ll_dg_3_1_c.STL; visual mesh filename=visual_stl/ll_dg_3_1.stl
- link ll_dg_3_2: geometry collision mesh filename=vendor_left/meshes/ll_dg_3_2_c.STL; visual mesh filename=visual_stl/ll_dg_3_2.stl
- link ll_dg_3_3: geometry collision mesh filename=vendor_left/meshes/ll_dg_3_3_c.STL; visual mesh filename=visual_stl/ll_dg_3_3.stl
- link ll_dg_3_4: geometry collision mesh filename=vendor_left/meshes/ll_dg_3_4_c.STL; visual mesh filename=visual_stl/ll_dg_3_4.stl
- link ll_dg_3_tip: geometry collision mesh filename=vendor_left/meshes/ll_dg_3_tip_c.STL; visual mesh filename=visual_stl/ll_dg_3_tip.stl
- link ll_dg_4_1: geometry collision mesh filename=vendor_left/meshes/ll_dg_4_1_c.STL; visual mesh filename=visual_stl/ll_dg_4_1.stl
- link ll_dg_4_2: geometry collision mesh filename=vendor_left/meshes/ll_dg_4_2_c.STL; visual mesh filename=visual_stl/ll_dg_4_2.stl
- link ll_dg_4_3: geometry collision mesh filename=vendor_left/meshes/ll_dg_4_3_c.STL; visual mesh filename=visual_stl/ll_dg_4_3.stl
- link ll_dg_4_4: geometry collision mesh filename=vendor_left/meshes/ll_dg_4_4_c.STL; visual mesh filename=visual_stl/ll_dg_4_4.stl
- link ll_dg_4_tip: geometry collision mesh filename=vendor_left/meshes/ll_dg_4_tip_c.STL; visual mesh filename=visual_stl/ll_dg_4_tip.stl
- link ll_dg_5_1: geometry collision mesh filename=vendor_left/meshes/ll_dg_5_1_c.STL; visual mesh filename=visual_stl/ll_dg_5_1.stl
- link ll_dg_5_2: geometry collision mesh filename=vendor_left/meshes/ll_dg_5_2_c.STL; visual mesh filename=visual_stl/ll_dg_5_2.stl
- link ll_dg_5_3: geometry collision mesh filename=vendor_left/meshes/ll_dg_5_3_c.STL; visual mesh filename=visual_stl/ll_dg_5_3.stl
- link ll_dg_5_4: geometry collision mesh filename=vendor_left/meshes/ll_dg_5_4_c.STL; visual mesh filename=visual_stl/ll_dg_5_4.stl
- link ll_dg_5_tip: geometry collision mesh filename=vendor_left/meshes/ll_dg_5_tip_c.STL; visual mesh filename=visual_stl/ll_dg_5_tip.stl
- link ll_dg_palm: geometry collision mesh filename=vendor_left/meshes/ll_dg_palm_c.STL; visual mesh filename=visual_stl/ll_dg_palm.stl
