Commit message: Uniform hands: canonical joint conventions (+ = flex toward the grasp point / spread toward +y, 0 = home)
make_uniform.py flips and re-zeroes joints so the same normalised target means the
same motion on every hand: a joint that moves its fingertip mostly sideways is a
spread joint (+ toward +y in the shared left-hand palm frame), anything else a flex
joint (+ moves the fingertip toward a grasp point 5 cm in front of the palm centre);
joints that only twist a straight finger are judged with the finger curled, as UHAS
does. Recorded in canonical_map.json; tests check every link lands where it did
under q_new = sign * q_vendor - offset. The joint viewer gets convention-check
buttons. Allegro's thumb sign corrected after a visual check.

Co-Authored-By: Claude Opus 5.5 (1M context) <noreply@anthropic.com>
Claude-Session: https://claude.ai/code/session_01VEjfLD7vkNCwPYPC2HsL71

File: assets/urdf/unified_dynamics_commercial_hands/allegro/allegro_left.urdf (robot description, URDF)
Before this commit: robot allegro_left, 23 links, 22 joints
Joints:
- joint joint_12_0: limit lower=0.263 upper=1.396 effort=0.5 velocity=10.0 -> lower=0 upper=1.133 effort=0.5 velocity=10.0; origin xyz=-0.0182 -0.019333 -0.045987 rpy=0 -1.65806278845 1.5707963259 -> xyz=-0.0182 -0.019333 -0.045987 rpy=-2.87859265 -1.48352987 -1.57079633

File: assets/urdf/unified_dynamics_commercial_hands/dex3/dex3_left.urdf (robot description, URDF)
Before this commit: robot dex3_1_l, 8 links, 7 joints
Joints:
- joint left_hand_index_0_joint: axis 0 0 1 -> -0 -0 -1; limit lower=-1.57079632 upper=0 effort=0.5 velocity=10.0 -> lower=-0 upper=1.57079632 effort=0.5 velocity=10.0
- joint left_hand_index_1_joint: axis 0 0 1 -> -0 -0 -1; limit lower=-1.74532925 upper=0 effort=0.5 velocity=10.0 -> lower=-0 upper=1.74532925 effort=0.5 velocity=10.0
- joint left_hand_middle_0_joint: axis 0 0 1 -> -0 -0 -1; limit lower=-1.57079632 upper=0 effort=0.5 velocity=10.0 -> lower=-0 upper=1.57079632 effort=0.5 velocity=10.0
- joint left_hand_middle_1_joint: axis 0 0 1 -> -0 -0 -1; limit lower=-1.74532925 upper=0 effort=0.5 velocity=10.0 -> lower=-0 upper=1.74532925 effort=0.5 velocity=10.0

File: assets/urdf/unified_dynamics_commercial_hands/leap/leap_left.urdf (robot description, URDF)
Before this commit: robot leap_left, 21 links, 20 joints
Joints:
- joint j0: axis 0 0 -1 -> -0 -0 1
- joint j12: axis 0 0 -1 -> -0 -0 1; limit lower=-2.094 upper=0.349 effort=0.5 velocity=10.0 -> lower=-0.349 upper=2.094 effort=0.5 velocity=10.0
- joint j13: axis 0 0 -1 -> -0 -0 1; limit lower=-2.443 upper=0.47 effort=0.5 velocity=10.0 -> lower=-0.47 upper=2.443 effort=0.5 velocity=10.0
- joint j14: limit lower=-1.20 upper=1.90 effort=0.5 velocity=10.0 -> lower=-1.2 upper=1.9 effort=0.5 velocity=10.0
- joint j4: axis 0 0 -1 -> -0 -0 1
- joint j8: axis 0 0 -1 -> -0 -0 1

File: assets/urdf/unified_dynamics_commercial_hands/shadow/shadow_left.urdf (robot description, URDF)
Before this commit: robot shadow_left, 30 links, 29 joints
Joints:
- joint FFJ1: limit lower=0 upper=1.57079632679 effort=0.5 velocity=10.0 -> lower=0 upper=1.57079633 effort=0.5 velocity=10.0
- joint FFJ2: limit lower=0 upper=1.57079632679 effort=0.5 velocity=10.0 -> lower=0 upper=1.57079633 effort=0.5 velocity=10.0
- joint FFJ3: limit lower=-0.261799387799 upper=1.57079632679 effort=0.5 velocity=10.0 -> lower=-0.261799388 upper=1.57079633 effort=0.5 velocity=10.0
- joint FFJ4: limit lower=-0.349065850399 upper=0.349065850399 effort=0.5 velocity=10.0 -> lower=-0.34906585 upper=0.34906585 effort=0.5 velocity=10.0
- joint LFJ1: limit lower=0 upper=1.57079632679 effort=0.5 velocity=10.0 -> lower=0 upper=1.57079633 effort=0.5 velocity=10.0
- joint LFJ2: limit lower=0 upper=1.57079632679 effort=0.5 velocity=10.0 -> lower=0 upper=1.57079633 effort=0.5 velocity=10.0
- joint LFJ3: limit lower=-0.261799387799 upper=1.57079632679 effort=0.5 velocity=10.0 -> lower=-0.261799388 upper=1.57079633 effort=0.5 velocity=10.0
- joint LFJ4: axis 0 -1 0 -> -0 1 -0; limit lower=-0.349065850399 upper=0.349065850399 effort=0.5 velocity=10.0 -> lower=-0.34906585 upper=0.34906585 effort=0.5 velocity=10.0
- joint LFJ5: limit lower=0 upper=0.785398163397 effort=0.5 velocity=10.0 -> lower=0 upper=0.785398163 effort=0.5 velocity=10.0
- joint MFJ1: limit lower=0 upper=1.57079632679 effort=0.5 velocity=10.0 -> lower=0 upper=1.57079633 effort=0.5 velocity=10.0
- joint MFJ2: limit lower=0 upper=1.57079632679 effort=0.5 velocity=10.0 -> lower=0 upper=1.57079633 effort=0.5 velocity=10.0
- joint MFJ3: limit lower=-0.261799387799 upper=1.57079632679 effort=0.5 velocity=10.0 -> lower=-0.261799388 upper=1.57079633 effort=0.5 velocity=10.0
- joint MFJ4: limit lower=-0.349065850399 upper=0.349065850399 effort=0.5 velocity=10.0 -> lower=-0.34906585 upper=0.34906585 effort=0.5 velocity=10.0
- joint RFJ1: limit lower=0 upper=1.57079632679 effort=0.5 velocity=10.0 -> lower=0 upper=1.57079633 effort=0.5 velocity=10.0
- joint RFJ2: limit lower=0 upper=1.57079632679 effort=0.5 velocity=10.0 -> lower=0 upper=1.57079633 effort=0.5 velocity=10.0
- joint RFJ3: limit lower=-0.261799387799 upper=1.57079632679 effort=0.5 velocity=10.0 -> lower=-0.261799388 upper=1.57079633 effort=0.5 velocity=10.0
- joint RFJ4: axis 0 -1 0 -> -0 1 -0; limit lower=-0.349065850399 upper=0.349065850399 effort=0.5 velocity=10.0 -> lower=-0.34906585 upper=0.34906585 effort=0.5 velocity=10.0
- joint THJ1: limit lower=-0.261799387799 upper=1.57079632679 effort=0.5 velocity=10.0 -> lower=-0.261799388 upper=1.57079633 effort=0.5 velocity=10.0
- joint THJ2: limit lower=-0.698131700798 upper=0.698131700798 effort=0.5 velocity=10.0 -> lower=-0.698131701 upper=0.698131701 effort=0.5 velocity=10.0
- joint THJ3: limit lower=-0.209439510239 upper=0.209439510239 effort=0.5 velocity=10.0 -> lower=-0.20943951 upper=0.20943951 effort=0.5 velocity=10.0
- joint THJ4: limit lower=0.0 upper=1.2217304764 effort=0.5 velocity=10.0 -> lower=0 upper=1.22173048 effort=0.5 velocity=10.0
- joint THJ5: limit lower=-1.0471975512 upper=1.0471975512 effort=0.5 velocity=10.0 -> lower=-1.04719755 upper=1.04719755 effort=0.5 velocity=10.0

File: assets/urdf/unified_dynamics_commercial_hands/sharpa/sharpa_left.urdf (robot description, URDF)
Before this commit: robot sharpa_left_unified, 33 links, 32 joints
Joints:
- joint left_5_pinky_CMC: axis 0 0 1 -> -0 -0 -1; limit lower=0 upper=0.2618 effort=0.5 velocity=10.0 -> lower=-0.2618 upper=-0 effort=0.5 velocity=10.0
- joint left_thumb_MCP_AA: axis 0 0 1 -> -0 -0 -1

File: assets/urdf/unified_dynamics_commercial_hands/tesollo/tesollo_left.urdf (robot description, URDF)
Before this commit: robot dg5f_left, 26 links, 25 joints
Joints:
- joint lj_dg_1_1: axis 1 0 0 -> -1 -0 -0; limit lower=-0.8901179185171081 upper=0.3839724354387525 effort=0.5 velocity=10.0 -> lower=-0.383972435 upper=0.890117919 effort=0.5 velocity=10.0
- joint lj_dg_1_2: limit lower=-0.0 upper=3.141592653589793 effort=0.5 velocity=10.0 -> lower=-0 upper=3.14159265 effort=0.5 velocity=10.0
- joint lj_dg_1_3: axis 1 0 0 -> -1 -0 -0; limit lower=-1.5707963267948966 upper=1.5707963267948966 effort=0.5 velocity=10.0 -> lower=-1.57079633 upper=1.57079633 effort=0.5 velocity=10.0
- joint lj_dg_1_4: axis 1 0 0 -> -1 -0 -0; limit lower=-1.5707963267948966 upper=1.5707963267948966 effort=0.5 velocity=10.0 -> lower=-1.57079633 upper=1.57079633 effort=0.5 velocity=10.0
- joint lj_dg_2_1: axis 1 0 0 -> -1 -0 -0; limit lower=-0.6108652381980153 upper=0.4188790204786391 effort=0.5 velocity=10.0 -> lower=-0.41887902 upper=0.610865238 effort=0.5 velocity=10.0
- joint lj_dg_2_2: limit lower=-0.0 upper=2.007128639793479 effort=0.5 velocity=10.0 -> lower=-0 upper=2.00712864 effort=0.5 velocity=10.0
- joint lj_dg_2_3: limit lower=-1.5707963267948966 upper=1.5707963267948966 effort=0.5 velocity=10.0 -> lower=-1.57079633 upper=1.57079633 effort=0.5 velocity=10.0
- joint lj_dg_2_4: limit lower=-1.5707963267948966 upper=1.5707963267948966 effort=0.5 velocity=10.0 -> lower=-1.57079633 upper=1.57079633 effort=0.5 velocity=10.0
- joint lj_dg_3_1: axis 1 0 0 -> -1 -0 -0; limit lower=-0.6108652381980153 upper=0.6108652381980153 effort=0.5 velocity=10.0 -> lower=-0.610865238 upper=0.610865238 effort=0.5 velocity=10.0
- joint lj_dg_3_2: limit lower=0.0 upper=1.9547687622336491 effort=0.5 velocity=10.0 -> lower=0 upper=1.95476876 effort=0.5 velocity=10.0
- joint lj_dg_3_3: limit lower=-1.5707963267948966 upper=1.5707963267948966 effort=0.5 velocity=10.0 -> lower=-1.57079633 upper=1.57079633 effort=0.5 velocity=10.0
- joint lj_dg_3_4: limit lower=-1.5707963267948966 upper=1.5707963267948966 effort=0.5 velocity=10.0 -> lower=-1.57079633 upper=1.57079633 effort=0.5 velocity=10.0
- joint lj_dg_4_1: axis 1 0 0 -> -1 -0 -0; limit lower=-0.4188790204786391 upper=0.6108652381980153 effort=0.5 velocity=10.0 -> lower=-0.610865238 upper=0.41887902 effort=0.5 velocity=10.0
- joint lj_dg_4_2: limit lower=0.0 upper=1.9024088846738192 effort=0.5 velocity=10.0 -> lower=0 upper=1.90240888 effort=0.5 velocity=10.0
- joint lj_dg_4_3: limit lower=-1.5707963267948966 upper=1.5707963267948966 effort=0.5 velocity=10.0 -> lower=-1.57079633 upper=1.57079633 effort=0.5 velocity=10.0
- joint lj_dg_4_4: limit lower=-1.5707963267948966 upper=1.5707963267948966 effort=0.5 velocity=10.0 -> lower=-1.57079633 upper=1.57079633 effort=0.5 velocity=10.0
- joint lj_dg_5_1: axis 0 0 1 -> -0 -0 -1; limit lower=-1.0471975511965976 upper=0.017453292519943295 effort=0.5 velocity=10.0 -> lower=-0.0174532925 upper=1.04719755 effort=0.5 velocity=10.0
- joint lj_dg_5_2: axis 1 0 0 -> -1 -0 -0; limit lower=-0.6108652381980153 upper=0.4188790204786391 effort=0.5 velocity=10.0 -> lower=-0.41887902 upper=0.610865238 effort=0.5 velocity=10.0
- joint lj_dg_5_3: limit lower=-1.5707963267948966 upper=1.5707963267948966 effort=0.5 velocity=10.0 -> lower=-1.57079633 upper=1.57079633 effort=0.5 velocity=10.0
- joint lj_dg_5_4: limit lower=-1.5707963267948966 upper=1.5707963267948966 effort=0.5 velocity=10.0 -> lower=-1.57079633 upper=1.57079633 effort=0.5 velocity=10.0

File: assets/urdf/unified_dynamics_commercial_hands/wuji2/wuji2_left.urdf (robot description, URDF)
Before this commit: robot wujihand2-beta2-left, 31 links, 30 joints
Joints:
- joint l_index_finger_dip: limit lower=-1.0470 upper=1.5700 effort=0.5 velocity=10.0 -> lower=-1.047 upper=1.57 effort=0.5 velocity=10.0
- joint l_index_finger_mcp_abd: limit lower=-0.6980 upper=0.6980 effort=0.5 velocity=10.0 -> lower=-0.698 upper=0.698 effort=0.5 velocity=10.0
- joint l_index_finger_mcp_flex: limit lower=-1.0470 upper=1.5700 effort=0.5 velocity=10.0 -> lower=-1.047 upper=1.57 effort=0.5 velocity=10.0
- joint l_index_finger_pip: limit lower=-1.0470 upper=2.0940 effort=0.5 velocity=10.0 -> lower=-1.047 upper=2.094 effort=0.5 velocity=10.0
- joint l_middle_finger_dip: limit lower=-1.0470 upper=1.5700 effort=0.5 velocity=10.0 -> lower=-1.047 upper=1.57 effort=0.5 velocity=10.0
- joint l_middle_finger_mcp_abd: limit lower=-0.6980 upper=0.6980 effort=0.5 velocity=10.0 -> lower=-0.698 upper=0.698 effort=0.5 velocity=10.0
- joint l_middle_finger_mcp_flex: limit lower=-1.0470 upper=1.5700 effort=0.5 velocity=10.0 -> lower=-1.047 upper=1.57 effort=0.5 velocity=10.0
- joint l_middle_finger_pip: limit lower=-1.0470 upper=2.0940 effort=0.5 velocity=10.0 -> lower=-1.047 upper=2.094 effort=0.5 velocity=10.0
- joint l_pinky_dip: limit lower=-1.0470 upper=1.5700 effort=0.5 velocity=10.0 -> lower=-1.047 upper=1.57 effort=0.5 velocity=10.0
- joint l_pinky_mcp_abd: limit lower=-0.6980 upper=0.6980 effort=0.5 velocity=10.0 -> lower=-0.698 upper=0.698 effort=0.5 velocity=10.0
- joint l_pinky_mcp_flex: limit lower=-1.0470 upper=1.5700 effort=0.5 velocity=10.0 -> lower=-1.047 upper=1.57 effort=0.5 velocity=10.0
- joint l_pinky_pip: limit lower=-1.0470 upper=2.0940 effort=0.5 velocity=10.0 -> lower=-1.047 upper=2.094 effort=0.5 velocity=10.0
- joint l_ring_finger_dip: limit lower=-1.0470 upper=1.5700 effort=0.5 velocity=10.0 -> lower=-1.047 upper=1.57 effort=0.5 velocity=10.0
- joint l_ring_finger_mcp_abd: limit lower=-0.6980 upper=0.6980 effort=0.5 velocity=10.0 -> lower=-0.698 upper=0.698 effort=0.5 velocity=10.0
- joint l_ring_finger_mcp_flex: limit lower=-1.0470 upper=1.5700 effort=0.5 velocity=10.0 -> lower=-1.047 upper=1.57 effort=0.5 velocity=10.0
- joint l_ring_finger_pip: limit lower=-1.0470 upper=2.0940 effort=0.5 velocity=10.0 -> lower=-1.047 upper=2.094 effort=0.5 velocity=10.0
- joint l_thumb_cmc_abd: limit lower=-1.4840 upper=0.6980 effort=0.5 velocity=10.0 -> lower=-1.484 upper=0.698 effort=0.5 velocity=10.0
- joint l_thumb_cmc_flex: limit lower=-1.1870 upper=1.2910 effort=0.5 velocity=10.0 -> lower=-1.187 upper=1.291 effort=0.5 velocity=10.0
- joint l_thumb_ip: limit lower=-1.0470 upper=1.5700 effort=0.5 velocity=10.0 -> lower=-1.047 upper=1.57 effort=0.5 velocity=10.0
- joint l_thumb_mcp: limit lower=-1.0470 upper=1.5700 effort=0.5 velocity=10.0 -> lower=-1.047 upper=1.57 effort=0.5 velocity=10.0
