Commit message: commercial.fit: the palm normal faces where the fingers flex; Allegro and MIDAS replicas were built back to front
_palm_axes took x = y cross z with y from the first row base to the last, so the vendor's digit order alone decided
whether x faced the grasp or the back of the hand. For Allegro and MIDAS it faced the back: the replicas were turned
180 degrees about the fingers, thumb opposing from the wrong side (Allegro: 42 mm cube spawn gap across the palm).
Digits now carry their URDF joint limits; x is flipped (with y, about z) when it opposes the flexion direction. All
four frames agree with onboarding's palm_frame; overlay base errors unchanged; 60/60 commercial tests pass.
Replicas regenerated.

Co-Authored-By: Claude Opus 5.5 <noreply@anthropic.com>
Claude-Session: https://claude.ai/code/session_01VEjfLD7vkNCwPYPC2HsL71

File: assets/urdf/unified_dynamics_commercial_hands_replicas/allegro/allegro_left_replica.urdf (robot description, URDF)
Before this commit: robot generated_hand, 31 links, 30 joints
Joints:
- joint f0_j0: origin xyz=-0.04829629131445342 -0.012940952255126037 0.14 rpy=-2.8797932657906435 -1.5707963267948966 0.0 -> xyz=0.04829629131445342 0.012940952255126037 0.14 rpy=-2.8797932657906435 -1.5707963267948966 0.0
- joint f1_j0: origin xyz=-0.004829629131445342 -0.0012940952255126037 0.14 rpy=-2.8797932657906435 -1.5707963267948966 0.0 -> xyz=0.004829629131445342 0.0012940952255126037 0.14 rpy=-2.8797932657906435 -1.5707963267948966 0.0
- joint f2_j0: origin xyz=0.038637033051562734 0.01035276180410083 0.14 rpy=-2.8797932657906435 -1.5707963267948966 0.0 -> xyz=-0.038637033051562734 -0.01035276180410083 0.14 rpy=-2.8797932657906435 -1.5707963267948966 0.0
- joint f3_j0: origin xyz=0.009659258262890684 0.0025881904510252074 0.065 rpy=3.141592653589793 0.0 0.26179938779914935 -> xyz=-0.009659258262890684 -0.0025881904510252074 0.065 rpy=0.0 2.220446049250313e-16 -2.8797932657906435
- joint f3_j1: origin xyz=0.05 0.0 0.0 rpy=0.0 0.0 -0.7853981633961052 -> xyz=0.05 0.0 -3.469446951953614e-18 rpy=0.0 0.0 0.7853981633961052
- joint f3_j2: origin xyz=0.020000000000000004 0.0 0.0 rpy=0.0 0.0 0.7853981633961052 -> xyz=0.020000000000000004 0.0 0.0 rpy=0.0 0.0 -0.7853981633961052
- joint f3_j3: origin xyz=0.05 0.0 0.0 rpy=0.0 0.0 -1.3652495408048331e-33 -> xyz=0.05 0.0 0.0 rpy=-3.4211388289180104e-49 0.0 1.3652495408048331e-33
- joint f3_j4: origin xyz=0.05500000000000001 0.0 0.0 rpy=0.0 0.0 -1.3652495408048331e-33 -> xyz=0.05500000000000001 0.0 -3.469446951953614e-18 rpy=-3.4211388289180104e-49 0.0 1.3652495408048331e-33

File: assets/urdf/unified_dynamics_commercial_hands_replicas/midas/midas_replica.urdf (robot description, URDF)
Before this commit: robot generated_hand, 31 links, 30 joints
Joints:
- joint f0_j0: origin xyz=-0.02897777478867205 -0.007764571353075622 0.13 rpy=-2.8797932657906435 -1.5707963267948966 0.0 -> xyz=0.02897777478867205 0.007764571353075622 0.13 rpy=-2.8797932657906435 -1.5707963267948966 0.0
- joint f1_j0: origin xyz=0.004829629131445342 0.0012940952255126037 0.14 rpy=-2.8797932657906435 -1.5707963267948966 0.0 -> xyz=-0.004829629131445342 -0.0012940952255126037 0.14 rpy=-2.8797932657906435 -1.5707963267948966 0.0
- joint f2_j0: origin xyz=0.038637033051562734 0.01035276180410083 0.13 rpy=-2.8797932657906435 -1.5707963267948966 0.0 -> xyz=-0.038637033051562734 -0.01035276180410083 0.13 rpy=-2.8797932657906435 -1.5707963267948966 0.0
- joint f3_j0: origin xyz=-0.019318516525781367 -0.005176380902050415 0.08 rpy=0.0 2.220446049250313e-16 -2.8797932657906435 -> xyz=0.019318516525781367 0.005176380902050415 0.08 rpy=3.141592653589793 0.0 0.26179938779914935
- joint f3_j1: origin xyz=0.019999999999999997 0.0 0.0 rpy=0.0 0.0 0.0 -> xyz=0.02 0.0 -1.734723475976807e-18 rpy=0.0 0.0 0.0
- joint f3_j2: origin xyz=0.060000000000000005 0.0 1.734723475976807e-18 rpy=0.0 -0.7853981633961051 0.0 -> xyz=0.060000000000000005 0.0 1.734723475976807e-18 rpy=0.0 0.7853981633961054 0.0
- joint f3_j3: origin xyz=0.04 0.0 -1.3877787807814457e-17 rpy=0.0 -0.7853981633961051 0.0 -> xyz=0.03999999999999998 0.0 0.0 rpy=0.0 0.7853981633961054 0.0
- joint f3_j4: origin xyz=0.030000000000000002 0.0 0.0 rpy=0.0 0.0 0.0 -> xyz=0.03 0.0 2.7755575615628914e-17 rpy=0.0 0.0 0.0

Commit message: commercial.fit: keep the vendor's joint direction (axis_override when the axis opposes the kind's default)
The kind fixes the hinge line; its sign was dropped ('an axis and its negative are the same hinge'), which turned
every Wuji v2 and LEAP abduction joint and LEAP's and Allegro's thumb joints the other way from the vendor's under
the same command (Wuji: 5/20 joints, LEAP 6/16, Allegro 3/16). A reversed axis now rides on axis_override, which
axis_of -- and so the sim build, the viewing URDF and FK -- honours. 0 reversed joints after; 88 tests pass.
Replicas regenerated.

Co-Authored-By: Claude Opus 5.5 <noreply@anthropic.com>
Claude-Session: https://claude.ai/code/session_01VEjfLD7vkNCwPYPC2HsL71

File: assets/urdf/unified_dynamics_commercial_hands_replicas/allegro/allegro_left_replica.urdf (robot description, URDF)
Before this commit: robot generated_hand, 31 links, 30 joints
Joints:
- joint f3_j1: axis 1.0 0.0 0.0 -> -1.0 -0.0 -0.0
- joint f3_j2: axis 0.0 1.0 0.0 -> -0.0 -1.0 -0.0
- joint f3_j3: axis 0.0 1.0 0.0 -> -0.0 -1.0 -0.0

File: assets/urdf/unified_dynamics_commercial_hands_replicas/leap/leap_left_replica.urdf (robot description, URDF)
Before this commit: robot generated_hand, 31 links, 30 joints
Joints:
- joint f0_j1: axis 0.0 1.0 0.0 -> -0.0 -1.0 -0.0
- joint f1_j1: axis 0.0 1.0 0.0 -> -0.0 -1.0 -0.0
- joint f2_j1: axis 0.0 1.0 0.0 -> -0.0 -1.0 -0.0
- joint f3_j1: axis 1.0 0.0 0.0 -> -1.0 -0.0 -0.0
- joint f3_j2: axis 0.0 1.0 0.0 -> -0.0 -1.0 -0.0
- joint f3_j3: axis 0.0 1.0 0.0 -> -0.0 -1.0 -0.0

File: assets/urdf/unified_dynamics_commercial_hands_replicas/midas/midas_replica.urdf (robot description, URDF)
Before this commit: robot generated_hand, 31 links, 30 joints
Joints:
- joint f0_j1: axis 0.0 0.0 1.0 -> -0.0 -0.0 -1.0
- joint f0_j2: axis 0.0 0.0 1.0 -> -0.0 -0.0 -1.0
- joint f0_j3: axis 0.0 0.0 1.0 -> -0.0 -0.0 -1.0
- joint f1_j1: axis 0.0 0.0 1.0 -> -0.0 -0.0 -1.0
- joint f1_j2: axis 0.0 0.0 1.0 -> -0.0 -0.0 -1.0
- joint f1_j3: axis 0.0 0.0 1.0 -> -0.0 -0.0 -1.0
- joint f2_j1: axis 0.0 0.0 1.0 -> -0.0 -0.0 -1.0
- joint f2_j2: axis 0.0 0.0 1.0 -> -0.0 -0.0 -1.0
- joint f2_j3: axis 0.0 0.0 1.0 -> -0.0 -0.0 -1.0
- joint f3_j1: axis 0.0 1.0 0.0 -> -0.0 -1.0 -0.0
- joint f3_j2: axis 0.0 0.0 1.0 -> -0.0 -0.0 -1.0
- joint f3_j3: axis 0.0 0.0 1.0 -> -0.0 -0.0 -1.0

File: assets/urdf/unified_dynamics_commercial_hands_replicas/wuji2/wuji2_left_replica.urdf (robot description, URDF)
Before this commit: robot generated_hand, 31 links, 30 joints
Joints:
- joint f0_j1: axis 0.0 1.0 0.0 -> -0.0 -1.0 -0.0
- joint f1_j1: axis 0.0 1.0 0.0 -> -0.0 -1.0 -0.0
- joint f2_j1: axis 0.0 1.0 0.0 -> -0.0 -1.0 -0.0
- joint f3_j1: axis 0.0 1.0 0.0 -> -0.0 -1.0 -0.0
- joint f4_j1: axis 0.0 1.0 0.0 -> -0.0 -1.0 -0.0
